File: 2-mill-vent/2-mill-vent.sch (KiCad schematic (older format))
At the start: 56 parts, among them J1 Differential:/Single, J3 No_Power_Control, J4 Front_panel_control, J5 Fan, J6 Ext Parts, J7 EXT Power Option, J8 POWER, Q1 2N3904, Q2 2N3904, Q3 2N3904, Q4 TSM480P06CHX0G-Transistor_FET, U1 LM358, U2 LM78L05_TO92, U3 TSR_1-24120, U4 MPXV

Commit message: Made major changes to 2A and started an all in one board
2A is a longer SMD front panel board now, no plans on updating 2b. work on 1, 2 , 2A, 2B has stoped.
Now looking at 3 to cut cost greatly with not having to interconnect two boards and make two boards. just the parts cost savings is in the order of $30 in qty1
Parts:
- removed A1: Arduino_Nano_v3.x, Module:Arduino_Nano, symbol 2-mill-vent-rescue:Arduino_Nano_v3.x-MCU_Module-1-mill-vent-rescue
- removed C10, C11, C9: 0.1uF, Capacitor_THT:C_Rect_L7.2mm_W2.5mm_P5.00mm_FKS2_FKP2_MKS2_MKP2, symbol Device:C_Small
- removed C5: 1uF, Capacitor_THT:CP_Radial_Tantal_D5.5mm_P2.50mm, symbol Device:CP1_Small
- removed D1: SW_Power, LED_THT:LED_D5.0mm, symbol Device:LED
- removed D2: +12V, LED_THT:LED_D5.0mm, symbol Device:LED
- removed D4: +5V, LED_THT:LED_D5.0mm, symbol Device:LED
- removed J1: Differential:/Single, Connector_PinHeader_2.54mm:PinHeader_1x03_P2.54mm_Vertical, symbol Connector:Conn_01x03_Male
- removed J3: No_Power_Control, Connector_PinHeader_2.54mm:PinHeader_1x02_P2.54mm_Vertical, symbol Connector:Conn_01x02_Male
- removed J6: Ext Parts, Connector_Molex:Molex_KK-254_AE-6410-05A_1x05_P2.54mm_Vertical, symbol Connector:Conn_01x05_Male
- removed J7: EXT Power Option, Connector_Molex:Molex_KK-254_AE-6410-04A_1x04_P2.54mm_Vertical, symbol Connector:Conn_01x04_Male
- removed Q1, Q2, Q3: 2N3904, Package_TO_SOT_THT:TO-92_Inline, symbol Transistor_BJT:2N3904
- removed R18: 1m, Resistor_THT:R_Axial_DIN0207_L6.3mm_D2.5mm_P2.54mm_Vertical, symbol Device:R_Small_US
- removed R20, R21, R22, R23, R24, R25, R26, R8: 330, Resistor_THT:R_Axial_DIN0207_L6.3mm_D2.5mm_P2.54mm_Vertical, symbol Device:R_Small_US
- removed R3: 1k, Resistor_THT:R_Axial_DIN0207_L6.3mm_D2.5mm_P2.54mm_Vertical, symbol Device:R_Small_US
- removed R7: 5k, Resistor_THT:R_Axial_DIN0207_L6.3mm_D2.5mm_P2.54mm_Vertical, symbol Device:R_Small_US
- removed R9: 10k, Resistor_THT:R_Axial_DIN0207_L6.3mm_D2.5mm_P2.54mm_Vertical, symbol Device:R_Small_US
- removed U1: LM358, Package_DIP:DIP-8_W7.62mm_Socket_LongPads, symbol Amplifier_Operational:LM358
- removed U2: LM78L05_TO92, Package_TO_SOT_THT:TO-92_Inline, symbol Regulator_Linear:LM78L05_TO92
- removed U4: MPXV, Sensor:MPXV, symbol 2-mill-vent-rescue:MPXV-Sensor-1-mill-vent-rescue
- added C1, C6: C0603C104M4RACTU, Capacitor_SMD:C_0603_1608Metric, symbol Device:C_Small
- added C3, C5: 1uF, Capacitor_THT:C_Rect_L7.2mm_W2.5mm_P5.00mm_FKS2_FKP2_MKS2_MKP2, symbol Device:C_Small
- added D2: 1N914, Diode_THT:D_DO-35_SOD27_P7.62mm_Horizontal, symbol Diode:1N914
- added J2: ICSP, Connector_PinHeader_2.54mm:PinHeader_2x03_P2.54mm_Vertical_SMD, symbol Connector_Generic:Conn_02x03_Odd_Even
- added J4: Buzzer, Connector_Molex:Molex_KK-254_AE-6410-03A_1x03_P2.54mm_Vertical, symbol Connector:Conn_01x03_Male
- added Q1, Q2, Q6: MMBT3904, Package_TO_SOT_SMD:SOT-23, symbol Transistor_BJT:MMBT3904
- added Q3, Q4: PZT3904, Package_TO_SOT_SMD:SOT-223-3_TabPin2, symbol Transistor_BJT:PZT3904
- added R14: 1M, Resistor_SMD:R_0603_1608Metric, symbol Device:R_Small_US
- added R2: 10k, Resistor_SMD:R_0603_1608Metric, symbol Device:R_Small_US
- added R7: 4814P-1-331LF, Package_SO:SOIC-14_3.9x8.7mm_P1.27mm, symbol Device:R_Pack07_SIP_Jim
- added U2: LM1117-5.0, Package_TO_SOT_SMD:TO-252-3_TabPin2, symbol Regulator_Linear:LM1117-5.0
- added U3: ATmega328P-AU, Package_QFP:TQFP-32_7x7mm_P0.8mm, symbol MCU_Microchip_ATmega:ATmega328P-AU
- added U4: LM321, Package_TO_SOT_SMD:SOT-23-5, symbol Amplifier_Operational:LM321
- added Y1: ABLS7M-16.000MHZ-B-2-T, Crystal:Crystal_SMD_7050-2Pin_7.0x5.0mm, symbol Device:Crystal_Small
- C2: renamed from C6; value 0.1uF -> C0603C104M4RACTU; footprint Capacitor_THT:C_Rect_L7.2mm_W2.5mm_P5.00mm_FKS2_FKP2_MKS2_MKP2 -> Capacitor_SMD:C_0603_1608Metric
- C4: value 10uF -> 1uF; footprint Capacitor_THT:C_Rect_L7.0mm_W3.5mm_P5.00mm -> Capacitor_THT:C_Rect_L7.2mm_W2.5mm_P5.00mm_FKS2_FKP2_MKS2_MKP2
- C7: value 0.1uF -> 10uF
- C8: value 470pF -> 1uF; footprint Capacitor_THT:C_Rect_L7.0mm_W3.5mm_P5.00mm -> Capacitor_THT:C_Rect_L7.2mm_W2.5mm_P5.00mm_FKS2_FKP2_MKS2_MKP2
- C9: renamed from C1; value 0.1uF -> C0603C104M4RACTU; footprint Capacitor_THT:C_Rect_L7.2mm_W2.5mm_P5.00mm_FKS2_FKP2_MKS2_MKP2 -> Capacitor_SMD:C_0603_1608Metric
- J1: renamed from J4; value Front_panel_control -> 71349-1006; footprint Connector_IDC:IDC-Header_2x08_P2.54mm_Vertical -> Connector_PinHeader_2.54mm:PinHeader_2x08_P2.54mm_Vertical_SMD
- Q5: renamed from Q4; value TSM480P06CHX0G-Transistor_FET -> TSM480P06CP; footprint Package_TO_SOT_THT:TO-251-3_Vertical -> Package_TO_SOT_SMD:TO-252-2
- R1: value 1.8k -> 10k; footprint Resistor_THT:R_Axial_DIN0207_L6.3mm_D2.5mm_P2.54mm_Vertical -> Resistor_SMD:R_0603_1608Metric
- R10: value 110 1W -> 10k; footprint Resistor_THT:R_Axial_DIN0617_L17.0mm_D6.0mm_P20.32mm_Horizontal -> Resistor_SMD:R_0603_1608Metric
- R11: renamed from R14; footprint Resistor_THT:R_Axial_DIN0207_L6.3mm_D2.5mm_P2.54mm_Vertical -> Resistor_SMD:R_0603_1608Metric
- R12: renamed from R17; footprint Resistor_THT:R_Axial_DIN0207_L6.3mm_D2.5mm_P2.54mm_Vertical -> Resistor_SMD:R_0603_1608Metric
- R13: renamed from R19; footprint Resistor_THT:R_Axial_DIN0207_L6.3mm_D2.5mm_P2.54mm_Vertical -> Resistor_SMD:R_0603_1608Metric
- R15: renamed from R28; footprint Resistor_THT:R_Axial_DIN0207_L6.3mm_D2.5mm_P2.54mm_Vertical -> Resistor_SMD:R_0603_1608Metric
- R16: renamed from R15; value 33k -> RN73H2ATTD3302D25; footprint Resistor_THT:R_Axial_DIN0207_L6.3mm_D2.5mm_P2.54mm_Vertical -> Resistor_SMD:R_0805_2012Metric
- R17: renamed from R16; value 8.2k -> RN73H2ATTD8201F25; footprint Resistor_THT:R_Axial_DIN0207_L6.3mm_D2.5mm_P2.54mm_Vertical -> Resistor_SMD:R_0805_2012Metric
- R3: renamed from R5; value 300 1/2W -> LTR18EZPJ301; footprint Resistor_THT:R_Axial_DIN0617_L17.0mm_D6.0mm_P20.32mm_Horizontal -> Resistor_SMD:R_1206_3216Metric_Pad1.42x1.75mm_HandSolder
- R4: value 10k -> 330; footprint Resistor_THT:R_Axial_DIN0207_L6.3mm_D2.5mm_P2.54mm_Vertical -> Resistor_SMD:R_0603_1608Metric
- R5: renamed from R27; value 1k -> 10k; footprint Resistor_THT:R_Axial_DIN0207_L6.3mm_D2.5mm_P2.54mm_Vertical -> Resistor_SMD:R_0603_1608Metric
- R6: value 10k -> 1k; footprint Resistor_THT:R_Axial_DIN0207_L6.3mm_D2.5mm_P2.54mm_Vertical -> Resistor_SMD:R_0603_1608Metric
- R8: renamed from R12; footprint Resistor_THT:R_Axial_DIN0207_L6.3mm_D2.5mm_P2.54mm_Vertical -> Resistor_SMD:R_0603_1608Metric
- R9: renamed from R2; footprint Resistor_THT:R_Axial_DIN0207_L6.3mm_D2.5mm_P2.54mm_Vertical -> Resistor_SMD:R_0603_1608Metric
- renumbered D3 to D1, J5 to J3, J8 to J5, U3 to U1
Connections:
- net Sensor_Power is gone; now on net +5V: C7.1
- net +12V: now also R13.2, C5.1, C6.1, R2.2, U2.3 (VI), U4.5 (V+); no longer C4.1, R10.2, R13.1
- net +5V: now also R1.2, R10.2, C1.2, J2.2 (Pin_2), U2.2 (VO), U3.18 (AVCC), U3.4 (VCC), U3.6 (VCC)
- net Batt_V: now also U4.3 (-), U4.4
- net Buzzer-: now also D1.2 (A), J4.3 (Pin_3), Q3.2 (C); no longer J1.10 (Pin_10)
- net Down: now also J2.1 (Pin_1), U3.16 (PB4)
- net GND: now also C1.1, C3.2, C5.2, C6.2, J2.6 (Pin_6), Q1.2 (E), Q2.2 (E), Q3.3 (E), Q4.3 (E), Q6.2 (E), U2.1 (GND), U3.21 (GND), U3.3 (GND), U3.5 (GND), U4.2 (V-); no longer R6.1
- net LED1: now also R7.8
- net LED2: now also R7.9
- net LED3: now also R7.10
- net LED5: now also R7.12
- net LED6: now also R7.13
- net LED7: now also R7.14 (-)
- net Motor+: now also J1.8 (Pin_8); no longer D1.1 (K)
- net Motor-: now also J1.10 (Pin_10), Q4.2 (C); no longer D1.2 (A)
- net ON\*OFF: now also C8.1, R13.1, Q6.1 (B), R14.2; no longer R13.2
- net PWM: now also R6.1; no longer J3.4 (Pin_4)
- net REF: now also U3.20 (AREF)
- net RPM: now also R1.1, Q1.3 (C); no longer R5.1
- net SW_Batt: now also D1.1 (K), J4.1 (Pin_1); no longer R1.1
- net Up: now also J2.4 (Pin_4), U3.15 (PB3)
- net at Q5.1 (G), R12.2: now also Q6.3 (C)
- net Raw_RPM: now reaches J3.3 (Pin_3), R15.1
- net Raw_RPM: now also R5.1; no longer R5.2
- net at R9.1: now also Q4.1 (B)
- net at J1.1 (Pin_1): now also R7.7
- net at J1.11 (Pin_11): now also R7.2
- net at J1.13 (Pin_13): now also R7.1
- net at J1.3 (Pin_3): now also R7.6
- net at J1.5 (Pin_5): now also R7.5
- net at J1.7 (Pin_7): now also R7.4
- net at J1.9 (Pin_9): now also R7.3
- net at R16.2, R17.1: now also U4.1 (+)
- net at R8.1: now also Q3.1 (B)
- net at R6.2: now also Q2.1 (B); no longer R4.2
- net Buzzer+ renamed Reset
- net Reset: now also J2.5 (Pin_5), U3.29 (~RESET~/PC6); no longer J1.8 (Pin_8)
- net Pressure: no longer names the net of R4.1
- net Pressure: now also Q2.3 (C), R2.1; no longer C8.1
- new net: Q1.1 (B), R5.2
- new net: C3.1, U3.7 (XTAL1/PB6), Y1.1
- new net: C4.1, U3.8 (XTAL2/PB7), Y1.2
- new net Error: R7.11
- new net Monitor: D2.2 (A), J2.3 (Pin_3), U3.17 (PB5)
- new net PWM_Drive: J3.4 (Pin_4), R4.2
- new net Power_off: D2.1 (K), R14.1
- no-connect marks 9 -> 1
Other:
- note added: "Buzzer:\nPin#3 Buzzer -\nPin#2 N/C\nPin#1 Buzzer +"
- note removed: "1597-1245-ND"
- note removed: "Arduino Nano\n V3 Board"
- note removed: "Ext. Parts:\nPin#5 Motor -\nPin#4 Motor +\nPin#3 +5v\nPin#2 Speed\nPin#1 Ground"
- note removed: "Note: A\n\nVoltage follower mode: \nR4 = 0k\nR6 = Open\nR7 = Open\nR9 = 0k\nJ1 1-2 = Open\nJ1 2-3 = Open\n\nNon-Inverting:\nR4 = 0K\nR6 = Open\nR7 = 10k\nR9 = 5k\nJ1 1-2 = Open\nJ1 2-3 = Closed\n\nDifferential:\nR19 = 10K\nR18 = 10K\nR17 = 10K\nR16 = 10K\nJ1 1-2 =Closed\nJ1 2-3 = Open\n\n"
- note removed: "Power Block: (MARKED BACKWARDS ON SILKSCREEN)\nPin#1 Switched Battery Voltage\nPin#2 +12V\nPin#3 +5V\nPin#4 Ground"
- note removed: "SEE Note: A"
- note removed: "TSM480P06CHX0G-ND"
- moved on the sheet: C2, C9, D1, F1, J1, J3, J5, Q5, R11, R12, R13, R15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
