File: 3-mill-vent/3-mill-vent.sch (KiCad schematic (older format))
At the start: 59 parts, among them J1 ICSP, J2 Fan, J3 Buzzer, J4 POWER, Q1 MMBT3904, Q2 MMBT3904, Q3 PZT3904, Q4 PZT3904, Q5 TSM480P06CP, Q6 MMBT3904, SW1 Power_off, SW2 Power_On, SW3 Fan_Down, SW4 Fan_Up, U1 ATmega328P-AU, U2 TSR_1-24120, U3 LM1117-5.0, U4 LM321, Y1 ABLS7M-16.000MHZ-B-2-T

Commit message: Just a check point
More work done on all in one board.
Now has step file of board with traces
Parts:
- added C7: LMK316AB7106MLHT, Capacitor_SMD:C_1206_3216Metric_Pad1.42x1.75mm_HandSolder, symbol Device:C_Small
- added D10, D12: FM4004-W, Diode_SMD:D_SMB, symbol Diode:1N4003
- added D13: D_Zener, symbol Device:D_Zener
- added R18: 47, Resistor_SMD:R_0603_1608Metric, symbol Device:R_Small_US
- C10: renamed from C3; value 1uF -> 1206Y0160180FFT; footprint Capacitor_THT:C_Rect_L7.2mm_W2.5mm_P5.00mm_FKS2_FKP2_MKS2_MKP2 -> Capacitor_SMD:C_1206_3216Metric
- C3: renamed from C6; value 1uF -> LMK316AB7106MLHT; footprint Capacitor_THT:C_Rect_L7.2mm_W2.5mm_P5.00mm_FKS2_FKP2_MKS2_MKP2 -> Capacitor_SMD:C_1206_3216Metric
- C5: renamed from C8; value 10uF -> T491C107M006AT; footprint Capacitor_THT:C_Rect_L7.2mm_W2.5mm_P5.00mm_FKS2_FKP2_MKS2_MKP2 -> Capacitor_Tantalum_SMD:CP_EIA-6032-15_Kemet-U
- C6: renamed from C9; footprint Capacitor_THT:C_Rect_L7.2mm_W2.5mm_P5.00mm_FKS2_FKP2_MKS2_MKP2 -> Capacitor_SMD:C_1206_3216Metric
- C9: renamed from C2; value 1uF -> 1206Y0160180FFT; footprint Capacitor_THT:C_Rect_L7.2mm_W2.5mm_P5.00mm_FKS2_FKP2_MKS2_MKP2 -> Capacitor_SMD:C_1206_3216Metric
- D11: renamed from D10; footprint Diode_THT:D_DO-35_SOD27_P7.62mm_Horizontal -> Diode_SMD:D_1206_3216Metric
- D7: value Fault -> Error
- D8: footprint Diode_THT:D_DO-35_SOD27_P7.62mm_Horizontal -> Diode_SMD:D_1206_3216Metric
- R14: renamed from R17; value RN73H2ATTD3302D25 -> RN73H2BTTD4702B10; footprint Resistor_SMD:R_0805_2012Metric -> Resistor_SMD:R_1206_3216Metric
- R17: renamed from R18; value RN73H2ATTD8201F25 -> RN73H2BTTD7061B10; footprint Resistor_SMD:R_0805_2012Metric -> Resistor_SMD:R_1206_3216Metric
- Y1: value ABLS7M-16.000MHZ-B-2-T -> 16.000MHZ; footprint Crystal:Crystal_SMD_7050-2Pin_7.0x5.0mm -> Crystal:Crystal_SMD_0603-2Pin_6.0x3.5mm
- renumbered C4 to C1, C5 to C2, C7 to C4, C1 to C8, R10 to R1, R13 to R10, R1 to R11, R2 to R12, R14 to R13, R16 to R15, R15 to R16, R3 to R19, R5 to R2, R19 to R20, R6 to R3, R7 to R4, R4 to R5, R8 to R6, R9 to R7, R11 to R8, R12 to R9, SW2 to SW1, SW3 to SW2, SW4 to SW3, SW1 to SW4, U2 to U1, U4 to U2, U1 to U4
Connections:
- net +12V: now also D10.1 (K)
- net +5V: now also C7.2, D12.1 (K); no longer C5.1, U3.2 (VO)
- net Batt_V: now also U4.22 (ADC7)
- net GND: now also C7.1, D13.2 (A), R18.1; no longer U3.1 (GND)
- net Monitor: now also D11.1 (K), U4.12 (PB0); no longer D11.2 (A)
- net Motor: now also U4.13 (PB1)
- net Raw_Batt: now also D13.1 (K)
- net at R15.2, SW1.1, SW4.2: now also D11.2 (A); no longer C6.1, Q6.1 (B), R16.1
- net at R15.1: now also C6.1, Q6.1 (B), R16.1; no longer D11.1 (K)
- new net: R18.2, U3.1 (GND)
- new net: C5.1, D10.2 (A), D12.2 (A), U3.2 (VO)
- no-connect marks 1 -> 2
Other:
- note added: "30V in 4.5V out\ndivided by 6.66"
- moved on the sheet: C1, C10, C2, C3, C4, C5, C6, C8, C9, D1, D11, D2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
