File: Older files/1-mill-vent/1-mill-vent.kicad_pcb (KiCad board)
At the start: 2 copper layers, 96.5 x 55.9 mm, 56 parts, among them J1 Differential:/Single, J3 No_Power_Control, J4 Front_panel_control, J5 Fan, J6 Ext Parts, J7 EXT Power Option, J8 POWER, Q1 2N3904, Q2 2N3904, Q3 2N3904, Q4 TSM480P06CHX0G-Transistor_FET, U1 LM358, U2 LM78L05_TO92, U3 TSR_1-24120, U4 MPXV

Commit message: last update for this round
last update for ver4 of board.
next will be ver5
Parts:
- moved C1 11.4 mm to (136.5, 115.6)
Routing:
- net ON\*OFF: track 84.9 -> 69.9 mm
- net GND: track 321.4 -> 310.3 mm, vias 68 -> 72
- net +12V: track 189.6 -> 190.9 mm
